File: pcb/8ch/expansion.sch (EAGLE design)
At the start: 56 parts, among them IC3 STM32F042F4, J7 AUDIO_JACK_3.5MM_PTH, J8 AUDIO_JACK_3.5MM_PTH, SW3 324_SW, SW4 324_SW, U1 USBC_16P, U2 USBC_16P, U4 XC6206_DEV

Commit message: added thermal on terminal block, adjusted terminal block and TRS connector location
Parts:
- U$14: device atx4vc:DG2204R-5.0-8DG2204-8 -> expansion:DG2204R-5.0-8DG2204-8
Changed lines of the file:
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@@
 <part name="R14" library="SparkFun-Passives" deviceset="RESISTOR" device="0805-RES" value="5K1"/>
 <part name="GND18" library="supply1" deviceset="GND" device=""/>
-<part name="U$14" library="atx4vc" deviceset="DG2204R-5.0-8" device="DG2204-8"/>
+<part name="U$14" library="expansion" deviceset="DG2204R-5.0-8" device="DG2204-8"/>
 <part name="J7" library="SparkFun-Connectors" deviceset="AUDIO_JACK_3.5MM" device="_PTH"/>
 <part name="J8" library="SparkFun-Connectors" deviceset="AUDIO_JACK_3.5MM" device="_PTH"/>
